File: door.kicad_pcb (KiCad board)
At the start: 2 copper layers, 100 x 85 mm, 32 parts, among them J1 Motor 1, J2 Motor 2, J3 POWER, J4 POWER, J5 Raspberry Pi Zero, J6 RC522 RFID Module, U1 DRV8838, U2 DRV8838, U3 SPX29302, U4 74HCT04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

Commit message: routing done
Parts:
- moved C11 174.9 mm to (60.2, 75.7), turned to 90 degrees
- moved C10 165.4 mm to (67.6, 75.7), turned to 90 degrees
- moved C9 157.9 mm to (76.5, 75.5), turned to 90 degrees
- moved C12 143.6 mm to (86.2, 72.8)
- moved C8 142.2 mm to (114.1, 80.1)
- moved R2 135.8 mm to (114.0, 76.3), turned to 180 degrees
- moved R1 130.3 mm to (114.0, 73.4)
- moved C3 128.3 mm to (114.0, 83.6)
- moved C2 120.6 mm to (137.3, 137.9)
- moved C6 111.2 mm to (137.3, 145.6), turned to 180 degrees
- moved C5 99.6 mm to (137.6, 128.8), turned to 180 degrees
- moved C1 95.7 mm to (137.5, 121.2)
- moved C4 13.1 mm to (130.6, 76.2)
- moved C7 5.68 mm to (122.0, 76.1), turned to 270 degrees
- moved U1 1.69 mm to (137.5, 125.2), turned to 180 degrees
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Connections:
- C5 pad 2: +5V -> /3V3_RASPI
- C6 pad 2: +5V -> /3V3_RASPI
- J5 pad 1: +5V -> /3V3_RASPI
- U1 pad 2: Net-(J1-Pad2) -> Net-(J1-Pad1)
- U1 pad 3: Net-(J1-Pad1) -> Net-(J1-Pad2)
- U1 pad 8: +5V -> /3V3_RASPI
- U2 pad 2: Net-(J2-Pad2) -> Net-(J2-Pad1)
- U2 pad 3: Net-(J2-Pad1) -> Net-(J2-Pad2)
- U2 pad 8: +5V -> /3V3_RASPI
Routing:
- net GND: track 0.00 -> 488.3 mm
- net +5V: track 0.00 -> 173.9 mm, vias 0 -> 2
- net +3V3: track 0.00 -> 132.5 mm, vias 0 -> 7
- net /3V3_RASPI: track 0.00 -> 89.8 mm, vias 0 -> 3
- net /RC522_RESET: track 0.00 -> 66.9 mm, vias 0 -> 1
- net /MISO: track 0.00 -> 62.6 mm, vias 0 -> 1
- net /MOSI: track 0.00 -> 60.2 mm, vias 0 -> 1
- net /SCLK: track 0.00 -> 59.1 mm, vias 0 -> 1
- net /CE0: track 0.00 -> 54.5 mm, vias 0 -> 1
- net /M2_EN: track 0.00 -> 52.4 mm
- net /M2_PH: track 0.00 -> 51.5 mm, vias 0 -> 1
- net /LED_DIN: track 0.00 -> 49.6 mm, vias 0 -> 2
- net /M2_nSLEEP: track 0.00 -> 44.8 mm, vias 0 -> 1
- net /M1_PH: track 0.00 -> 43.0 mm, vias 0 -> 1
- net Net-(F1-Pad2): track 0.00 -> 40.6 mm
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Other:
- net class Default: clearance 0.2 -> 0.16; trace_width 0.2 -> 0.25
- net class Power: clearance 0.3 -> 0.16; trace_width 0.5 -> 0.25
- rule trace_clearance: 0.2 -> 0.16

Commit message: almost done...
Parts:
- added REF***: Polarity_Center_Positive_6mm_SilkScreen, Symbols:Polarity_Center_Positive_6mm_SilkScreen, F.Cu at (116.1, 102.1)
Connections:
- U1 pad 9: (no net) -> GND
- U2 pad 9: (no net) -> GND
Routing:
- net +3V3: track 132.5 -> 139.0 mm
- net GND: track 488.3 -> 491.2 mm, vias 0 -> 7
- added copper zone on B.Cu, net GND
- added copper zone on F.Cu, net GND
Other:
- board text added: "+"
- board text added: "-"
- board text added: "5V DC INPUT"
- board text added: "M1"
- board text added: "M2"
- board text added: "RC522 RFID Module"
- board text added: "Raspberry Pi Zero"

Commit message: added schmatic pdf
Parts:
- added REF***: KiCad-Logo2_8mm_SilkScreen, Symbols:KiCad-Logo2_8mm_SilkScreen, B.Cu at (130.0, 145.0)
Other:
- board text added: "Tobias Kaiser 24 Feb 2018 door_pcb"

Commit message: fertig; PCBs bei seeedstudio bestellt
Parts:
- added J7: To current sense module, Pin_Headers:Pin_Header_Straight_1x10_Pitch2.54mm, B.Cu at (135.9, 151.2)
- added R3: 0, Resistors_SMD:R_1812_HandSoldering, F.Cu at (131.4, 117.2)
- added R4: 0, Resistors_SMD:R_1812_HandSoldering, F.Cu at (131.2, 133.3)
- U1, U2: footprint Housings_DFN_QFN:DFN-8-1EP_2x2mm_Pitch0.5mm -> Morn_SMD_NoLeads:DFN-8-1EP_2x2mm_Pitch0.5mm_FIXED
- moved REF*** 41.2 mm to (88.9, 148.6)
Connections:
- C1 pad 1: +3V3 -> /m1_csl
- C2 pad 1: +3V3 -> /m2_csl
- J5 pad 26: Net-(J5-Pad26) -> /CE1
- U1 pad 1: +3V3 -> /m1_csl
- U2 pad 1: +3V3 -> /m2_csl
Routing:
- net GND: track 491.2 -> 963.5 mm, vias 7 -> 39
- net +5V: track 173.9 -> 272.6 mm, vias 2 -> 4
- net /m1_csl: track 0.00 -> 53.4 mm, vias 0 -> 3
- net /MOSI: track 60.2 -> 110.0 mm
- net /SCLK: track 59.1 -> 97.4 mm
- net /m2_csl: track 0.00 -> 35.5 mm, vias 0 -> 3
- net /CE1: track 0.00 -> 32.4 mm
- net /MISO: track 62.6 -> 94.9 mm, vias 1 -> 2
- net +3V3: track 139.0 -> 153.8 mm, vias 7 -> 5
- net /3V3_RASPI: track 89.8 -> 102.3 mm
- net /M2_PH: track 51.5 -> 48.3 mm
- net /M2_nSLEEP: track 44.8 -> 46.7 mm
- net /M2_EN: track 52.4 -> 51.6 mm
Other:
- net class Default: clearance 0.16 -> 0.1524
- net class Power: clearance 0.16 -> 0.1524
- rule trace_clearance: 0.16 -> 0.1524
- board text added: "Tobias Kaiser 26 Feb 2018 door_pcb"
- board text removed: "Tobias Kaiser 24 Feb 2018 door_pcb"
